Commit message: fix: 修复夹爪单指运动问题（Gazebo 不执行 URDF mimic，改双指同步驱动）
根因：Gazebo Harmonic 运行时不支持 mimic 约束（gz-sim#1684），
fp3_finger_joint2 成为无约束、无命令的自由关节。

改动：
- panda.urdf.xacro：finger_joint2 增加 position 命令接口 + 状态接口
- panda_controllers.yaml：双指均入 joint_state_broadcaster /
  fp3_gripper_controller，补 gains，加 allow_partial_joints_goal
- panda.srdf：声明 <mimic_joint> 保持 MoveIt 1-DOF 规划语义
- hand_grasp_test.py / pick_place_full.py：轨迹同时驱动双指
- README / docs：更新说明，新增《夹爪单指运动问题修复记录.md》

实测验证：hand_grasp_test 双指全程同步；pick_place_full 成功
将物块从 z=0.115 夹起悬空至 z=0.212。

File: src/panda_grasp_sim/urdf/panda.urdf.xacro (robot description, xacro)
@@ -27,5 +27,7 @@
     <!--
         5. ros2_control 硬件接口配置
-           fp3_finger_joint2 是 mimic 关节，不应在此声明 command_interface
+           注意：两个手指关节都声明 command_interface，由控制器同步驱动。
+           Gazebo Harmonic 不执行 URDF mimic 约束（见 docs/gazebo_troubleshooting.md 坑 5），
+           MoveIt 侧通过在 panda.srdf 中声明 mimic_joint 保持 1-DOF 规划语义。
     -->
     <ros2_control name="PandaSimSystem" type="system">
@@ -62,4 +64,14 @@
             <state_interface name="effort"/>
         </joint>
+        <joint name="fp3_finger_joint2">
+            <command_interface name="position" />
+            <state_interface name="position">
+                <param name="initial_value">0.04</param>
+            </state_interface>
+            <state_interface name="velocity">
+                <param name="initial_value">0.0</param>
+            </state_interface>
+            <state_interface name="effort"/>
+        </joint>
     </ros2_control>
     <!-- 6. Gazebo 插件配置 -->
